Commit message: camera: use Gemini names across no-arm profile

File: urdf/ranger_mini.urdf (robot description, URDF)
Before this commit: robot ranger_mini_v2, 7 links, 6 joints
Links:
- added link camera_gemini330_link
Joints:
- added joint base_to_camera_gemini330: type fixed, parent base_link, child camera_gemini330_link, origin xyz=0.28 0 0.30 rpy=0 0 0
